File: kicad_files/project/voltage_supervisor.kicad_sch (KiCad schematic)
At the start: 2 parts, among them U8 MCP1319MT-29LE-OT

Commit message: misc: simplifiy power pins and other components, add test pins
Other:
- title: (none) -> Voltage Supervisor
Changed lines of the file:
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@@
 	(paper "A4")
 	(title_block
+		(title "Voltage Supervisor")
 		(date "2024-05-30")
 		(rev "0.1")
