File: hardware/kicad_files/project/logos.kicad_sch (KiCad schematic)
At the start: 1 part, among them T1 LOGO

Commit message: feat: add logos
Parts:
- added T2: LOGO, Logos:carl_zeiss_stiftung, symbol carl_zeiss_logo:LOGO
- added T3: LOGO, Logos:FORTE_logo_square, symbol FORTE_logo_square:LOGO
- added T4: LOGO, Logos:heidelberg-university-logo, symbol heidelberg-university-logo:LOGO
- added T5: LOGO, Logos:ukripluslogo, symbol ukriplus_logo:LOGO
- T1: footprint FABulous:fabulous_logo_qr_code_generated_30mm -> FABulous:fabulous_logo_qr_code_generated_25mm

Commit message: fix D2 LED orientation and change Pads of USB-C connector to avoid warnings, also exlude all logos from BOM
Parts:
- T3, T4, T5: now left out of the parts list
Changed lines of the file:
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@@
 		(unit 1)
 		(exclude_from_sim no)
-		(in_bom yes)
+		(in_bom no)
 		(on_board yes)
 		(dnp no)
@@
 		(unit 1)
 		(exclude_from_sim no)
-		(in_bom yes)
+		(in_bom no)
 		(on_board yes)
 		(dnp no)
@@
 		(unit 1)
 		(exclude_from_sim no)
-		(in_bom yes)
+		(in_bom no)
 		(on_board yes)
 		(dnp no)

Commit message: fix: replace all local symbols and footprints with versions from KiCad or project libraries
Parts:
- T1: footprint FABulous:fabulous_logo_qr_code_generated_25mm -> Logos:fabulous_logo_qr_code_generated_25mm; symbol FABulousLogo:LOGO -> logos:FABulous; now in the parts list
- T2: symbol carl_zeiss_logo:LOGO -> logos:carl_zeiss; now in the parts list
- T3: symbol FORTE_logo_square:LOGO -> logos:FORTE; now in the parts list
- T4: symbol heidelberg-university-logo:LOGO -> logos:heidelberg_university; now in the parts list
- T5: symbol ukriplus_logo:LOGO -> logos:UKRI; now in the parts list
Other:
- title: (none) -> Logos
Changed lines of the file:
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@@
 	(paper "A4")
 	(title_block
+		(title "Logos")
 		(date "2024-05-30")
 		(rev "0.1")
 	)
 	(symbol
-		(lib_id "FORTE_logo_square:LOGO")
+		(lib_id "logos:FORTE")
 		(at 134.62 83.82 0)
 		(unit 1)
 		(exclude_from_sim no)
-		(in_bom no)
+		(in_bom yes)
 		(on_board yes)
 		(dnp no)
@@
 	)
 	(symbol
-		(lib_id "carl_zeiss_logo:LOGO")
+		(lib_id "logos:carl_zeiss")
 		(at 123.19 83.82 0)
 		(unit 1)
 		(exclude_from_sim no)
-		(in_bom no)
+		(in_bom yes)
 		(on_board yes)
 		(dnp no)
@@
 	)
 	(symbol
-		(lib_id "ukriplus_logo:LOGO")
+		(lib_id "logos:UKRI")
 		(at 189.23 85.09 0)
 		(unit 1)
 		(exclude_from_sim no)
-		(in_bom no)
+		(in_bom yes)
 		(on_board yes)
 		(dnp no)
@@
 	)
 	(symbol
-		(lib_id "heidelberg-university-logo:LOGO")
+		(lib_id "logos:heidelberg_university")
 		(at 156.21 83.82 0)
 		(unit 1)
 		(exclude_from_sim no)
-		(in_bom no)
+		(in_bom yes)
 		(on_board yes)
 		(dnp no)
@@
 	)
 	(symbol
-		(lib_name "LOGO_1")
-		(lib_id "FABulousLogo:LOGO")
+		(lib_id "logos:FABulous")
 		(at 102.87 86.36 0)
 		(unit 1)
 		(exclude_from_sim no)
-		(in_bom no)
+		(in_bom yes)
 		(on_board yes)
 		(dnp no)
@@
 			)
 		)
-		(property "Footprint" "FABulous:fabulous_logo_qr_code_generated_25mm"
+		(property "Footprint" "Logos:fabulous_logo_qr_code_generated_25mm"
 			(at 102.87 86.36 0)
 			(effects
