File: hardware/kicad_files/project/test_points.kicad_sch (KiCad schematic)
At the start: 4 parts

Commit message: feat: Implement all findings of the second review
Parts:
- TP1, TP2, TP3, TP4: now left out of the parts list
Changed lines of the file:
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@@
 		(unit 1)
 		(exclude_from_sim no)
-		(in_bom yes)
+		(in_bom no)
 		(on_board yes)
 		(dnp no)
@@
 		(on_board yes)
 		(dnp no)
-		(property "Reference" "#PWR082"
+		(property "Reference" "#PWR084"
 			(at 146.05 100.33 0)
 			(effects
@@
 			(project "FABulous_board"
 				(path "/5664f05e-a3ef-4177-8026-c4580fa32c71/238deadf-4ea7-42f0-993c-dcd1bd51f50c"
-					(reference "#PWR082")
+					(reference "#PWR084")
 					(unit 1)
 				)
@@
 		(dnp no)
 		(fields_autoplaced yes)
-		(property "Reference" "#PWR081"
+		(property "Reference" "#PWR083"
 			(at 135.89 100.33 0)
 			(effects
@@
 			(project "FABulous_board"
 				(path "/5664f05e-a3ef-4177-8026-c4580fa32c71/238deadf-4ea7-42f0-993c-dcd1bd51f50c"
-					(reference "#PWR081")
+					(reference "#PWR083")
 					(unit 1)
 				)
@@
 		(dnp no)
 		(fields_autoplaced yes)
-		(property "Reference" "#PWR083"
+		(property "Reference" "#PWR085"
 			(at 156.21 100.33 0)
 			(effects
@@
 			(project "FABulous_board"
 				(path "/5664f05e-a3ef-4177-8026-c4580fa32c71/238deadf-4ea7-42f0-993c-dcd1bd51f50c"
-					(reference "#PWR083")
+					(reference "#PWR085")
 					(unit 1)
 				)
@@
 		(unit 1)
 		(exclude_from_sim no)
-		(in_bom yes)
+		(in_bom no)
 		(on_board yes)
 		(dnp no)
@@
 		(unit 1)
 		(exclude_from_sim no)
-		(in_bom yes)
+		(in_bom no)
 		(on_board yes)
 		(dnp no)
@@
 		(unit 1)
 		(exclude_from_sim no)
-		(in_bom yes)
+		(in_bom no)
 		(on_board yes)
 		(dnp no)
@@
 		(dnp no)
 		(fields_autoplaced yes)
-		(property "Reference" "#PWR080"
+		(property "Reference" "#PWR082"
 			(at 125.73 107.95 0)
 			(effects
@@
 			(project "FABulous_board"
 				(path "/5664f05e-a3ef-4177-8026-c4580fa32c71/238deadf-4ea7-42f0-993c-dcd1bd51f50c"
-					(reference "#PWR080")
-					(unit 1)
-				)
+					(reference "#PWR082")
+					(unit 1)
+				)
